Commit message: lotsa updates

File: description/lidar.xacro (robot description, xacro)
@@ -22,9 +22,9 @@
         </xacro:inertial_cylinder>
     </link>
-    <gazebo reference="laser_frame">
+    <gazebo reference="laser_frame">  <!-- Must mat ch the link name we are going to work on-->
         <material>Gazebo/Red</material>
-        <sensor name="laser" type="ray">
-            <pose>0 0 0 0 0 0</pose>
-            <visualize>true</visualize>
+        <sensor name="laser" type="ray">   <!-- The Name here doens't matter but the type MUST be "ray" -->
+            <pose>0 0 0 0 0 0</pose>       <!-- This is the origin in reference to the origin of the link we apply this to. -->
+            <visualize>true</visualize>    <!-- Allows us to turn this on/off with code maybe? -->
             <update_rate>10</update_rate>
             <ray>
@@ -41,4 +41,5 @@
                 </range>
             </ray>
+            <!--  This section is the executeable plugin for gazebo to allow us to generate test data -->
             <plugin name="laser_controller" filename="libgazebo_ros_ray_sensor.so">
                 <ros>

File: description/robot.urdf.xacro (robot description, xacro)
@@ -1,8 +1,17 @@
 <?xml version="1.0"?>
 <robot xmlns:xacro="http://www.ros.org/wiki/xacro"  name="robot">
+<!-- This file is going to be used to setup our robot. -->
+<!-- It does not contain any description. -->
+<!-- Description compondents are added as individual includes -->
+    <!-- This is our robot base and minimum viable description -->
+    <!-- Do NOT comment this include out or we will not have a robot. -->
     <xacro:include filename="robot_core.xacro" />
-    <!-- <xacro:include filename="gazebo_control.xacro" /> -->
-    <!-- Note that we cannot (I believe use bot gazebo_control and ros2_control at the same time.) -->
+    <!-- Load the description file for the Lidar.  Can be commented out to disable -->
+    <xacro:include filename="lidar.xacro" />
+    <!-- Load the description file for the camera.  Can be commented out to disable -->
+    <xacro:include filename="camera.xacro" />
+    <!-- Load the control module for Gazebo -->
+    <xacro:include filename="gazebo_control.xacro" />
+    <!-- Note that we cannot (I believe) use both gazebo_control and ros2_control at the same time. -->
     <xacro:include filename="ros2_control.xacro" />
-    <!-- <xacro:include filename="lidar.xacro" /> -->
 </robot>

File: description/robot_core.xacro (robot description, xacro)
@@ -46,62 +46,4 @@
         <material>Gazebo/White</material>
     </gazebo>
-<!-- test -->
-<!--
-    <joint name="arm_joint" type="continuous">
-        <parent link="base_link"/>
-        <child link="arm_link"/>
-        <origin xyz="0 1 0"/>
-        <axis xyz="0 1 0"/>
-    </joint>
-    <link name="arm_link">
-        <visual>
-            <origin xyz="0.15 0.5 0.075" />
-            <geometry>
-                <box size="0.1 0.3 0.1" />
-            </geometry>
-            <material name="white" />
-        </visual>
-        <collision>
-            <origin xyz="0.15 0.5 0.075" />
-            <geometry>
-                <box size="0.1 0.3 0.1" />
-            </geometry>
-        </collision>
-        <xacro:inertial_box mass="0.5" x="0.3" y="0.3" z="0.15">
-            <origin xyz="0.15 0.0 0.075" rpy="0.0 0.0 0.0"/>
-        </xacro:inertial_box>
-    </link>
-    <gazebo reference="arm_link">
-        <material>Gazebo/White</material>
-    </gazebo>
-    <joint name="arm_joint2" type="continuous">
-        <parent link="arm_link"/>
-        <child link="arm_link2"/>
-        <origin xyz="0 0.0 0"/>
-        <axis xyz="0 1 0"/>
-    </joint>
-    <link name="arm_link2">
-        <visual>
-            <origin xyz="0.15 1 0.075" />
-            <geometry>
-                <box size="0.1 0.3 0.1" />
-            </geometry>
-            <material name="white" />
-        </visual>
-        <collision>
-            <origin xyz="0.15 1 0.075" />
-            <geometry>
-                <box size="0.1 0.3 0.1" />
-            </geometry>
-        </collision>
-        <xacro:inertial_box mass="0.5" x="0.3" y="0.3" z="0.15">
-            <origin xyz="0.15 1 0.075" rpy="0.0 0.0 0.0"/>
-        </xacro:inertial_box>
-    </link>
-    <gazebo reference="arm_link2">
-        <material>Gazebo/White</material>
-    </gazebo>
-    -->
-<!-- end test -->
     <!-- Left Wheel Link -->
     <joint name="left_wheel_joint" type="continuous">
