Commit message: various updates

File: description/camera.xacro (robot description, xacro)
@@ -1,49 +1,39 @@
 <?xml version="1.0"?>
-<robot xmlns:xacro="http://www.ros.org/wiki/xacro">
+<robot xmlns:xacro="http://www.ros.org/wiki/xacro" >
+    <!-- Additional plugins to install when using a camera -->
+    <!-- sudo apt install ros-humble-image-transport-plugins -->
+    <!-- sudo apt install ros-humble-rqt-image-view -->
+    <!-- sudo apt install v4l-utils ros-humble-v4l2-camera -->
+    <!-- Extra informaiton on this file here: https://www.youtube.com/watch?v=A3nw2M47K50&list=PLunhqkrRNRhYAffV8JDiFOatQXuU-NnxT&index=10 -->
     <joint name="camera_joint" type="fixed">
         <parent link="chassis"/>
         <child link="camera_link"/>
-        <origin xyz="0.305 0.0 0.8" rpy="0.0 0.0 0.0"/>
+        <origin xyz="0.305 0 0.08" rpy="0 0 0"/>
     </joint>
     <link name="camera_link">
         <visual>
             <geometry>
-                <box size="0.010 0.03 0.03 "/>
+                <box size="0.010 0.03 0.03"/>
             </geometry>
-            <material name="red" />
+            <material name="red"/>
         </visual>
-        <collision>
-            <geometry>
-                <box size="0.010 0.03 0.03 "/>
-            </geometry>
-        </collision>
-        <xacro:inertial_cylinder mass="0.1" length="0.04" radius="0.05">
-            <origin xyz="0.0 0.0 0.0" rpy="0.0 0.0 0.0"/>
-        </xacro:inertial_cylinder>
     </link>
-    <!-- This is a special joint and link for gazebo -->
     <joint name="camera_optical_joint" type="fixed">
         <parent link="camera_link"/>
         <child link="camera_link_optical"/>
-        <origin xyz="0 0 0" rpy="${-pi/2} 0.0 ${-pi/2}"/>
+        <origin xyz="0 0 0" rpy="${-pi/2} 0 ${-pi/2}"/>
     </joint>
-    <link name="camera_link_optical"> </link>
-    <!-- End special gazebo joint and link -->
-    <gazebo reference="laser_frame">  <!-- Must mat ch the link name we are going to work on-->
+    <link name="camera_link_optical"></link>
+    <gazebo reference="camera_link">
         <material>Gazebo/Red</material>
-        <!-- The Name here doens't matter but the type MUST be "ray" -->
-        <sensor name="laser" type="ray">
-            <!-- This is the origin in reference to the origin of the link we apply this to. -->
-            <pose>0 0 0 0 0 0</pose>
-            <!-- Allows us to turn this on/off with code maybe? -->
+        <sensor name="camera" type="camera">
+            <pose> 0 0 0 0 0 0 </pose>
             <visualize>true</visualize>
             <update_rate>10</update_rate>
-            <!-- These are the properties of the physical camera -->
-            <!-- Can also be the properties of the virtual gazebo camera  -->
             <camera>
                 <horizontal_fov>1.089</horizontal_fov>
                 <image>
-                    <format>R8G8B8</format> <!-- 8 bits of each color -->
-                    <width>640</width> <!-- Size of the camera resolution -->
+                    <format>R8G8B8</format>
+                    <width>640</width>
                     <height>480</height>
                 </image>
@@ -53,7 +43,6 @@
                 </clip>
             </camera>
-            <!--  This section is the executeable plugin for gazebo to allow us to generate test data -->
             <plugin name="camera_controller" filename="libgazebo_ros_camera.so">
-                <frame_name>camera_link_optical_frame</frame_name>
+                <frame_name>camera_link_optical</frame_name>
             </plugin>
         </sensor>
