Commit message: current build

File: description/robot.urdf.xacro (robot description, xacro)
@@ -2,3 +2,5 @@
 <robot xmlns:xacro="http://www.ros.org/wiki/xacro"  name="robot">
     <xacro:include filename="robot_core.xacro" />
+    <xacro:include filename="gazebo_control.xacro" />
+    <xacro:include filename="lidar.xacro" />
 </robot>

File: description/robot_core copy.xacro (robot description, xacro)
@@ -46,32 +46,4 @@
         <material>Gazebo/White</material>
     </gazebo>
-<!-- test -->
-    <!-- <joint name="arm_joint" type="fixed">
-        <parent link="chassis"/>
-        <child link="arm_link"/>
-        <origin xyz="-0.1 1 0"/>
-    </joint>
-    <link name="arm_link">
-        <visual>
-            <origin xyz="0.15 1 0.075" />
-            <geometry>
-                <box size="0.1 1.3 0.1" />
-            </geometry>
-            <material name="white" />
-        </visual>
-        <collision>
-            <origin xyz="0.15 1 0.075" />
-            <geometry>
-                <box size="0.1 1.3 0.1" />
-            </geometry>
-        </collision>
-        <xacro:inertial_box mass="0.5" x="0.3" y="0.3" z="0.15">
-            <origin xyz="0.15 1.0 0.075" rpy="0.0 0.0 0.0"/>
-        </xacro:inertial_box>
-    </link>
-    <gazebo reference="arm_link">
-        <material>Gazebo/White</material>
-    </gazebo> -->
-<!-- end test -->
     <!-- Left Wheel Link -->
     <joint name="left_wheel_joint" type="continuous">

Commit message: upload changes

File: description/robot.urdf.xacro (robot description, xacro)
@@ -3,4 +3,4 @@
     <xacro:include filename="robot_core.xacro" />
     <xacro:include filename="gazebo_control.xacro" />
-    <xacro:include filename="lidar.xacro" />
+    <!-- <xacro:include filename="lidar.xacro" /> -->
 </robot>

File: description/robot_core.xacro (robot description, xacro)
@@ -47,14 +47,43 @@
     </gazebo>
 <!-- test -->
-    <!-- <joint name="arm_joint" type="fixed">
-        <parent link="chassis"/>
+<!--
+    <joint name="arm_joint" type="continuous">
+        <parent link="base_link"/>
         <child link="arm_link"/>
-        <origin xyz="-0.1 1 0"/>
+        <origin xyz="0 1 0"/>
+        <axis xyz="0 1 0"/>
     </joint>
     <link name="arm_link">
         <visual>
+            <origin xyz="0.15 0.5 0.075" />
+            <geometry>
+                <box size="0.1 0.3 0.1" />
+            </geometry>
+            <material name="white" />
+        </visual>
+        <collision>
+            <origin xyz="0.15 0.5 0.075" />
+            <geometry>
+                <box size="0.1 0.3 0.1" />
+            </geometry>
+        </collision>
+        <xacro:inertial_box mass="0.5" x="0.3" y="0.3" z="0.15">
+            <origin xyz="0.15 0.0 0.075" rpy="0.0 0.0 0.0"/>
+        </xacro:inertial_box>
+    </link>
+    <gazebo reference="arm_link">
+        <material>Gazebo/White</material>
+    </gazebo>
+    <joint name="arm_joint2" type="continuous">
+        <parent link="arm_link"/>
+        <child link="arm_link2"/>
+        <origin xyz="0 0.0 0"/>
+        <axis xyz="0 1 0"/>
+    </joint>
+    <link name="arm_link2">
+        <visual>
             <origin xyz="0.15 1 0.075" />
             <geometry>
-                <box size="0.1 1.3 0.1" />
+                <box size="0.1 0.3 0.1" />
             </geometry>
             <material name="white" />
@@ -63,14 +92,15 @@
             <origin xyz="0.15 1 0.075" />
             <geometry>
-                <box size="0.1 1.3 0.1" />
+                <box size="0.1 0.3 0.1" />
             </geometry>
         </collision>
         <xacro:inertial_box mass="0.5" x="0.3" y="0.3" z="0.15">
-            <origin xyz="0.15 1.0 0.075" rpy="0.0 0.0 0.0"/>
+            <origin xyz="0.15 1 0.075" rpy="0.0 0.0 0.0"/>
         </xacro:inertial_box>
     </link>
-    <gazebo reference="arm_link">
+    <gazebo reference="arm_link2">
         <material>Gazebo/White</material>
-    </gazebo> -->
+    </gazebo>
+    -->
 <!-- end test -->
     <!-- Left Wheel Link -->

Commit message: Many changes

File: description/robot.urdf.xacro (robot description, xacro)
@@ -4,17 +4,23 @@
 <!-- It does not contain any description. -->
 <!-- Description compondents are added as individual includes -->
+    <!-- These two parameters state if we are using gazzebo or hardware control -->
+    <!-- I don't believe I can use both -->
+    <xacro:arg name="use_ros2_control" default="true"/>
+    <xacro:arg name="sim_mode" default="false"/>
     <!-- This is our robot base and minimum viable description -->
     <!-- Do NOT comment this include out or we will not have a robot. -->
     <xacro:include filename="robot_core.xacro" />
+    <!-- These are to enable ros2control or gazebo control when needed. -->
+    <!-- For now I am going to do it manually.-->
+    <xacro:if value="$(arg use_ros2_control)">
+        <xacro:include filename="ros2_control.xacro" />
+    </xacro:if>
+    <xacro:unless value="$(arg use_ros2_control)">
+        <xacro:include filename="gazebo_control.xacro" />
+    </xacro:unless>
     <!-- Load the description file for the Lidar.  Can be commented out to disable -->
     <xacro:include filename="lidar.xacro" />
     <!-- Load the description file for the camera.  Can be commented out to disable -->
     <xacro:include filename="camera.xacro" />
-    <!-- Load the control module for Gazebo -->
-    <!-- Without this line our robot won't move in gazebo when given commands -->
-    <!-- with ex. teleop_twist_keyboard -->
-    <!-- August 28/23, we are going to disable this for the hardware ros2_control below -->
-    <!-- <xacro:include filename="gazebo_control.xacro" /> -->
-    <!-- Note that we cannot (I believe) use both gazebo_control and ros2_control at the same time. -->
-    <xacro:include filename="ros2_control.xacro" />
+    <!-- <xacro:include filename="depth_camera.xacro" /> -->
 </robot>

File: description/ros2_control.xacro (robot description, xacro)
@@ -1,46 +1,61 @@
 <?xml version="1.0"?>
 <robot xmlns:xacro="http://www.ros.org/wiki/xacro">
-    <ros2_control name="GazeboSystem" type="system">
-        <hardware>
-            <!-- this plugin is our *hardware* interface -->
-            <!-- later we will add a gazebo tag for its interface -->
-            <!-- in this case tells ros2_controll how to talk to gazebo -->
-            <!-- as if it was talking to real hardware -->
-            <plugin>gazebo_ros2_control/GazeboSystem</plugin>
-        </hardware>
-        <!-- We need to define each interface with a ros2_control interface -->
-        <!-- A command_interface is what is going to receive numbers to act upon -->
-        <!-- state_interface is what we can read to see what the current state is -->
-        <joint name="left_wheel_joint">
-            <command_interface name="velocity">
-                <param name="min">-10</param>
-                <param name="max">10</param>
-            </command_interface>
-            <state_interface name="velocity"/>
-            <state_interface name="position"/>
-        </joint>
-        <joint name="right_wheel_joint">
-            <command_interface name="velocity">
-                <param name="min">-10</param>
-                <param name="max">10</param>
-            </command_interface>
-            <state_interface name="velocity"/>
-            <state_interface name="position"/>
-        </joint>
-    </ros2_control>
+    <xacro:unless value="$(arg sim_mode)">
+        <ros2_control name="RealRobot" type="system">
+            <hardware>
+                <plugin>diffdrive_arduino/DiffDriveArduino</plugin>
+                <param name="left_wheel_name">left_wheel_joint</param>
+                <param name="right_wheel_name">right_wheel_joint</param>
+                <param name="loop_rate">30</param>
+                <param name="device">/dev/ttyUSB0</param>
+                <param name="baud_rate">57600</param>
+                <param name="timeout">1000</param>
+                <param name="enc_counts_per_rev">3436</param>
+            </hardware>
+            <joint name="left_wheel_joint">
+                <command_interface name="velocity">
+                    <param name="min">-10</param>
+                    <param name="max">10</param>
+                </command_interface>
+                <state_interface name="velocity"/>
+                <state_interface name="position"/>
+            </joint>
+            <joint name="right_wheel_joint">
+                <command_interface name="velocity">
+                    <param name="min">-10</param>
+                    <param name="max">10</param>
+                </command_interface>
+                <state_interface name="velocity"/>
+                <state_interface name="position"/>
+            </joint>
+        </ros2_control>
+    </xacro:unless>
+    <xacro:if value="$(arg sim_mode)">
+        <ros2_control name="GazeboSystem" type="system">
+            <hardware>
+                <plugin>gazebo_ros2_control/GazeboSystem</plugin>
+            </hardware>
+            <joint name="left_wheel_joint">
+                <command_interface name="velocity">
+                    <param name="min">-10</param>
+                    <param name="max">10</param>
+                </command_interface>
+                <state_interface name="velocity"/>
+                <state_interface name="position"/>
+            </joint>
+            <joint name="right_wheel_joint">
+                <command_interface name="velocity">
+                    <param name="min">-10</param>
+                    <param name="max">10</param>
+                </command_interface>
+                <state_interface name="velocity"/>
+                <state_interface name="position"/>
+            </joint>
+        </ros2_control>
+    </xacro:if>
     <gazebo>
-    <!-- This plugin recieves the cmd_vel from joint_state_publisher and -->
-    <!-- translates them into gazebo movements. -->
-    <!-- name= is not specific.  any identifier is fine and is arbitrary -->
-    <!-- filename= is important and is the file name of the plugin -->
-    <!-- In this inst ance we are starting the gazebo_ros2_control plugin -->
-    <!-- when not using gazebo, we will need to run "ros2 run controller_manager ros2_control_node" -->
-    <!-- It contains its own control manager -->
-    <!-- It gets most of its other setup from the robot_state_publisher but not for the ros2_control system -->
-    <!-- It has been noted in video  https://www.youtube.com/watch?v=4QKsDf1c4hc&list=PLunhqkrRNRhYAffV8JDiFOatQXuU-NnxT&index=12 -->
-    <!--   that when not using gazebo, we need to run -->
-    <!--   ros2 run controller_manager ros2_ccontrol_node     Investigate further -->
         <plugin name="gazebo_ros2_control" filename="libgazebo_ros2_control.so">
-            <parameters>$(find inmoov_base)/config/controllers.yaml</parameters>
+            <parameters>$(find inmoov_base)/config/my_controllers.yaml</parameters>
+            <parameters>$(find inmoov_base)/config/gaz_ros2_ctl_use_sim.yaml</parameters>
         </plugin>
     </gazebo>

Commit message: commit a bunch of changes

File: description/robot.urdf.xacro (robot description, xacro)
@@ -1,17 +1,19 @@
 <?xml version="1.0"?>
-<robot xmlns:xacro="http://www.ros.org/wiki/xacro"  name="robot">
+<robot xmlns:xacro="http://www.ros.org/wiki/xacro"  name="inmoov">
     <xacro:arg name="use_ros2_control" default="true"/>
     <xacro:arg name="sim_mode" default="false"/>
     <xacro:include filename="robot_core.xacro" />
-    <xacro:if value="$(arg use_ros2_control)">
+    <!-- <xacro:if value="$(arg use_ros2_control)">
         <xacro:include filename="ros2_control.xacro" />
     </xacro:if>
     <xacro:unless value="$(arg use_ros2_control)">
         <xacro:include filename="gazebo_control.xacro" />
-    </xacro:unless>
-    <xacro:include filename="lidar.xacro" />
-    <xacro:include filename="camera.xacro" />
+    </xacro:unless> -->
+    <!-- <xacro:include filename="lidar.xacro" /> -->
+    <!-- <xacro:include filename="camera.xacro" /> -->
     <!-- <xacro:include filename="depth_camera.xacro" /> -->
     <xacro:include filename="face.xacro" />
-    <xacro:include filename="inmoov.urdf.xacro" />
+    <!-- This is for my robot to attach to the top of the base.   -->
+    <!-- For now we don't need it -->
+    <!-- <xacro:include filename="inmoov.urdf.xacro" /> -->
 </robot>

File: description/robot_core.xacro (robot description, xacro)
@@ -2,4 +2,7 @@
 <robot xmlns:xacro="http://www.ros.org/wiki/xacro" >
     <xacro:include filename="inertial_macros.xacro"/>
+    <xacro:include filename="robot_gazebo.xacro"/>
+    <!-- Pi Constant -->
+    <!-- <xacro:property name="pi" value="3.14159"/> -->
     <xacro:property name="chassis_length" value="0.335"/>
     <xacro:property name="chassis_width" value="0.265"/>
@@ -32,21 +35,33 @@
     </material>
     <!-- BASE LINK -->
+    <!-- I believe this is what is linking to the world
+    but that is yet to come -->
+<!--
     <link name="base_link">
-    </link>
+    </link> -->
     <!-- BASE_FOOTPRINT LINK -->
-<!--
-    <joint name="base_footprint_joint" type="fixed">
-        <parent link="base_link"/>
-        <child link="base_footprint"/>
-        <origin xyz="0 0 0" rpy="0 0 0"/>
+    <!-- This was required for the newer version of gazebo.
+        It expects to see a "base_footprint" link that is attached
+        to some other link on our robot.  Base Link in our case.
+        It will be attached with a "base_footprint_joint".
+        I believe it is somewhat synonymous to the world link
+        that was commonly used in previous versions of gazebo
+    -->
+    <link name="base_footprint"></link>
+    <joint name="base_link_joint" type="fixed">
+        <parent link="base_footprint"/>
+        <child link="chassis"/>
+        <!-- <origin xyz="0 0 0" rpy="0 0 0"/> -->
+        <!-- I am going ot use the wheel link offsets from before -->
+        <origin xyz="${-wheel_offset_x} 0 ${-wheel_offset_z}"/>
     </joint>
-    <link name="base_footprint">
-    </link> -->
     <!-- CHASSIS LINK -->
-    <joint name="chassis_joint" type="fixed">
+    <!-- since changing to the base_footprint model for the -->
+    <!-- more recent versions of gazebo, we don't need this link -->
+    <!-- <joint name="chassis_joint" type="fixed">
         <parent link="base_link"/>
         <child link="chassis"/>
         <origin xyz="${-wheel_offset_x} 0 ${-wheel_offset_z}"/>
-    </joint>
+    </joint> -->
     <link name="chassis">
         <visual>
@@ -67,7 +82,4 @@
         </xacro:inertial_box>
     </link>
-    <gazebo reference="chassis">
-        <material>Gazebo/Orange</material>
-    </gazebo>
     <!-- LEFT WHEEL LINK -->
     <joint name="left_wheel_joint" type="continuous">
@@ -93,7 +105,4 @@
         </xacro:inertial_cylinder>
     </link>
-    <gazebo reference="left_wheel">
-        <material>Gazebo/Blue</material>
-    </gazebo>
     <!-- RIGHT WHEEL LINK -->
     <joint name="right_wheel_joint" type="continuous">
@@ -103,5 +112,5 @@
         <axis xyz="0 0 -1"/>
     </joint>
-    <link name="right_wheel">
+    <link name="rigt_hwheel">
         <visual>
             <geometry>
@@ -119,7 +128,4 @@
         </xacro:inertial_cylinder>
     </link>
-    <gazebo reference="right_wheel">
-        <material>Gazebo/Blue</material>
-    </gazebo>
     <!-- CASTER WHEEL LINK -->
     <joint name="caster_wheel_joint" type="fixed">
@@ -144,8 +150,3 @@
         </xacro:inertial_sphere>
     </link>
-    <gazebo reference="caster_wheel">
-        <material>Gazebo/White</material>
-        <mu1 value="0.001"/>
-        <mu2 value="0.001"/>
-    </gazebo>
 </robot>
