Commit message: changes

File: description/robot_core.xacro (robot description, xacro)
@@ -2,16 +2,30 @@
 <robot xmlns:xacro="http://www.ros.org/wiki/xacro" >
     <material name="white">
-        <color rbga"1 1 1 1" />
+        <color rbga="1 1 1 1"/>
     </material>
     <material name="orange">
-        <color rbga"1 0.3 0.1 1" />
+        <color rbga="1 0.3 0.1 1"/>
     </material>
     <material name="blue">
-        <color rbga"0.2 0.2 1 1" />
+        <color rbga="0.2 0.2 1 1"/>
     </material>
     <material name="black">
-        <color rbga"0 0 0 1" />
+        <color rbga="0 0 0 1"/>
     </material>
     <link name="base_link">
     </link>
+    <joint name="chassis_joint" type="fixed">
+        <parent link="base_link"/>
+        <child link="chassis"/>
+        <origin xyz="-0.1 0 0"/>
+    </joint>
+    <link name="chassis">
+        <visual>
+            <origin xyz="0.15 0 0.075" />
+            <geometry>
+                <box size="0.3 0.3 0.15" />
+            </geometry>
+            <!-- <material name="white" /> -->
+        </visual>
+    </link>
 </robot>

Commit message: launcher changes

File: description/robot_core.xacro (robot description, xacro)
@@ -2,15 +2,16 @@
 <robot xmlns:xacro="http://www.ros.org/wiki/xacro" >
     <material name="white">
-        <color rbga="1 1 1 1"/>
+        <color rgba="1.0 1.0 1.0 1.0"/>
     </material>
     <material name="orange">
-        <color rbga="1 0.3 0.1 1"/>
+        <color rgba="1.0 1.0 1.0 1.0"/>
     </material>
     <material name="blue">
-        <color rbga="0.2 0.2 1 1"/>
+        <color rgba="0.2 0.2 1 1"/>
     </material>
     <material name="black">
-        <color rbga="0 0 0 1"/>
+        <color rgba="0 0 0 1"/>
     </material>
+    <!-- Base Link  -->
     <link name="base_link">
     </link>
@@ -26,6 +27,73 @@
                 <box size="0.3 0.3 0.15" />
             </geometry>
-            <!-- <material name="white" /> -->
+            <material name="white" />
         </visual>
+        <collision>
+            <origin xyz="0.15 0 0.075" />
+            <geometry>
+                <box size="0.3 0.3 0.15" />
+            </geometry>
+        </collision>
+    </link>
+    <!-- Left Wheel Link -->
+    <joint name="left_wheel_joint" type="continuous">
+        <parent link="base_link"/>
+        <child link="left_wheel"/>
+        <origin xyz="0.0 0.175 0.0" rpy="-${pi/2} 0.0 0.0"/>
+        <axis xyz="0.0 0.0 1.0"/>
+    </joint>
+    <link name="left_wheel">
+        <visual>
+            <geometry>
+                <cylinder radius="0.05" length="0.04"/>
+            </geometry>
+            <material name="blue" />
+        </visual>
+        <collision>
+            <geometry>
+                <cylinder radius="0.05" length="0.04"/>
+            </geometry>
+        </collision>
+    </link>
+    <!-- Right Wheel Link -->
+    <joint name="right_wheel_joint" type="continuous">
+        <parent link="base_link"/>
+        <child link="right_wheel"/>
+        <origin xyz="0.0 -0.175 0.0" rpy="${pi/2} 0 0"/>
+        <axis xyz="0.0 0.0 -1.0"/>
+    </joint>
+    <link name="right_wheel">
+        <visual>
+            <geometry>
+                <cylinder radius="0.05" length="0.04"/>
+            </geometry>
+            <material name="blue" />
+        </visual>
+        <collision>
+            <geometry>
+                <cylinder radius="0.05" length="0.04"/>
+            </geometry>
+        </collision>
+    </link>
+    <!-- Caster Wheel Link -->
+    <joint name="caster_wheel_joint" type="fixed">
+        <origin xyz="0.24 0.0 0.0" rpy="0.0 0.0 0.0"/>
+        <parent link="chassis"/>
+        <child link="caster_wheel"/>
+        <axis xyz="0.0 0.0 0.0"/>
+    </joint>
+    <link name="caster_wheel">
+        <visual name="">
+            <geometry>
+               <sphere radius="0.05"/>
+            </geometry>
+            <material name="black" />
+        </visual>
+        <collision name="">
+            <geometry>
+               <sphere radius="0.05"/>
+            </geometry>
+            <material name="black" />
+        </collision>
     </link>
 </robot>

Commit message: update

File: description/robot_core.xacro (robot description, xacro)
@@ -36,4 +36,7 @@
             </geometry>
         </collision>
+        <xacro:inertial_box mass="0.5" x="0.3" y="0.3" z="0.15">
+            <origin xyz="0.15 0.0 0.075" rpy="0.0 0.0 0.0"/>
+        </xacro:inertial_box>
     </link>
     <!-- Left Wheel Link -->
@@ -56,4 +59,7 @@
             </geometry>
         </collision>
+        <xacro:inertial_cylinder mass="0.1" length="0.04" radius="0.05">
+            <origin xyz="0.0 0.0 0.0" rpy="0.0 0.0 0.0"/>
+        </xacro:inertial_cylinder>
     </link>
     <!-- Right Wheel Link -->
@@ -76,4 +82,7 @@
             </geometry>
         </collision>
+        <xacro:inertial_cylinder mass="0.1" length="0.04" radius="0.05">
+            <origin xyz="0.0 0.0 0.0" rpy="0.0 0.0 0.0"/>
+        </xacro:inertial_cylinder>
     </link>
     <!-- Caster Wheel Link -->
@@ -97,4 +106,7 @@
             <material name="black" />
         </collision>
+        <xacro:inertial_sphere mass="0.1" radius="0.05">
+            <origin xyz="0.0 0.0" rpy="0.0 0.0 0.0"/>
+        </xacro:inertial_sphere>
     </link>
 </robot>

Commit message: TYPO

File: description/robot_core.xacro (robot description, xacro)
@@ -112,5 +112,5 @@
         <axis xyz="0 0 -1"/>
     </joint>
-    <link name="rigt_hwheel">
+    <link name="right_wheel">
         <visual>
             <geometry>
